File: robarm_pcb/motor_driver/motor_driver_prj/motor_connectors.sch (KiCad schematic (older format))
At the start: 1 part

Commit message: save
Parts:
- gave numbers to parts that had none: 1
Changed lines of the file:
@@
 $Descr A4 11693 8268
 encoding utf-8
-Sheet 3 15
+Sheet 8 15
 Title ""
 Date ""
@@
 P 5200 2900
 AR Path="/60338EBB/6032DB81" Ref="J?"  Part="1"
-AR Path="/60338EBB/6032D419/6032DB81" Ref="J?"  Part="1"
-AR Path="/60338EBB/603307A0/6032DB81" Ref="J?"  Part="1"
-AR Path="/60338EBB/60330C16/6032DB81" Ref="J?"  Part="1"
-AR Path="/60338EBB/603314BA/6032DB81" Ref="J?"  Part="1"
-AR Path="/60338EBB/60331A7A/6032DB81" Ref="J?"  Part="1"
-AR Path="/60338EBB/60331E19/6032DB81" Ref="J?"  Part="1"
-F 0 "J?" H 5308 3181 50  0000 C CNN
+AR Path="/60338EBB/6032D419/6032DB81" Ref="J3"  Part="1"
+AR Path="/60338EBB/603307A0/6032DB81" Ref="J4"  Part="1"
+AR Path="/60338EBB/60330C16/6032DB81" Ref="J5"  Part="1"
+AR Path="/60338EBB/603314BA/6032DB81" Ref="J6"  Part="1"
+AR Path="/60338EBB/60331A7A/6032DB81" Ref="J7"  Part="1"
+AR Path="/60338EBB/60331E19/6032DB81" Ref="J8"  Part="1"
+F 0 "J8" H 5308 3181 50  0000 C CNN
 F 1 "Conn_01x04_Male" H 5308 3090 50  0000 C CNN
 F 2 "Connector_Phoenix_MSTB:PhoenixContact_MSTBVA_2,5_4-G-5,08_1x04_P5.08mm_Vertical" H 5200 2900 50  0001 C CNN
