File: robarm_pcb/motor_driver/motor_driver_prj/AllDrivers.sch (KiCad schematic (older format))
At the start: 15 parts, among them U2 TCA9539PWR, U3 TCA9539PWR, U4 TCA9539PWR

Commit message: save
Parts:
- renumbered R8 to R10, R9 to R11, R10 to R12, R11 to R13, R12 to R14, R13 to R15, R14 to R16, R15 to R17, R4 to R6, R5 to R7, R6 to R8, R7 to R9, U2 to U5, U3 to U6, U4 to U7
Changed lines of the file:
@@
 $Descr A4 11693 8268
 encoding utf-8
-Sheet 3 15
+Sheet 9 15
 Title ""
 Date ""
@@
 P 3350 5850
 AR Path="/60365972" Ref="U?"  Part="1"
-AR Path="/603463D6/60365972" Ref="U3"  Part="1"
-F 0 "U3" H 3350 6965 50  0000 C CNN
+AR Path="/603463D6/60365972" Ref="U6"  Part="1"
+F 0 "U6" H 3350 6965 50  0000 C CNN
 F 1 "TCA9539PWR" H 3350 6874 50  0000 C CNN
 F 2 "motor_driver:TCA9539_TSSOP-24" H 3250 5550 50  0001 C CNN
@@
 P 3350 2400
 AR Path="/6036597E" Ref="U?"  Part="1"
-AR Path="/603463D6/6036597E" Ref="U2"  Part="1"
-F 0 "U2" H 3350 3515 50  0000 C CNN
+AR Path="/603463D6/6036597E" Ref="U5"  Part="1"
+F 0 "U5" H 3350 3515 50  0000 C CNN
 F 1 "TCA9539PWR" H 3350 3424 50  0000 C CNN
 F 2 "motor_driver:TCA9539_TSSOP-24" H 3250 2100 50  0001 C CNN
@@
 RRef4
 $Comp
-L power:VCC #PWR04
+L power:VCC #PWR023
 U 1 1 6036E484
 P 2100 1350
-F 0 "#PWR04" H 2100 1200 50  0001 C CNN
+F 0 "#PWR023" H 2100 1200 50  0001 C CNN
 F 1 "VCC" H 2115 1523 50  0000 C CNN
 F 2 "" H 2100 1350 50  0001 C CNN
@@
 	2100 1350 2100 1550
 $Comp
-L Device:R_Small_US R4
+L Device:R_Small_US R6
 U 1 1 60323950
 P 2200 1700
-F 0 "R4" H 2268 1700 50  0000 L CNN
+F 0 "R6" H 2268 1700 50  0000 L CNN
 F 1 "1" H 2268 1655 50  0001 L CNN
 F 2 "Resistor_SMD:R_0603_1608Metric_Pad0.98x0.95mm_HandSolder" H 2200 1700 50  0001 C CNN
@@
 $EndComp
 $Comp
-L Device:R_Small_US R6
+L Device:R_Small_US R8
 U 1 1 60327792
 P 2450 1800
-F 0 "R6" H 2518 1800 50  0000 L CNN
+F 0 "R8" H 2518 1800 50  0000 L CNN
 F 1 "1" H 2518 1755 50  0001 L CNN
 F 2 "Resistor_SMD:R_0603_1608Metric_Pad0.98x0.95mm_HandSolder" H 2450 1800 50  0001 C CNN
@@
 $EndComp
 $Comp
-L Device:R_Small_US R8
+L Device:R_Small_US R10
 U 1 1 6032E2C9
 P 2600 2200
-F 0 "R8" H 2668 2200 50  0000 L CNN
+F 0 "R10" H 2668 2200 50  0000 L CNN
 F 1 "1" H 2668 2155 50  0001 L CNN
 F 2 "Resistor_SMD:R_0603_1608Metric_Pad0.98x0.95mm_HandSolder" H 2600 2200 50  0001 C CNN
@@
 $EndComp
 $Comp
-L Device:R_Small_US R10
+L Device:R_Small_US R12
 U 1 1 60334C6F
 P 2800 2200
-F 0 "R10" H 2868 2200 50  0000 L CNN
+F 0 "R12" H 2868 2200 50  0000 L CNN
 F 1 "1" H 2868 2155 50  0001 L CNN
 F 2 "Resistor_SMD:R_0603_1608Metric_Pad0.98x0.95mm_HandSolder" H 2800 2200 50  0001 C CNN
@@
 P 7950 2400
 AR Path="/60365978" Ref="U?"  Part="1"
-AR Path="/603463D6/60365978" Ref="U4"  Part="1"
-F 0 "U4" H 7950 3515 50  0000 C CNN
+AR Path="/603463D6/60365978" Ref="U7"  Part="1"
+F 0 "U7" H 7950 3515 50  0000 C CNN
 F 1 "TCA9539PWR" H 7950 3424 50  0000 C CNN
 F 2 "motor_driver:TCA9539_TSSOP-24" H 7850 2100 50  0001 C CNN
@@
 Connection ~ 2600 2450
 $Comp
-L power:GND #PWR08
+L power:GND #PWR027
 U 1 1 60406059
 P 2650 3400
-F 0 "#PWR08" H 2650 3150 50  0001 C CNN
+F 0 "#PWR027" H 2650 3150 50  0001 C CNN
 F 1 "GND" H 2655 3227 50  0000 C CNN
 F 2 "" H 2650 3400 50  0001 C CNN
@@
 	2650 3250 2650 3400
 $Comp
-L power:VCC #PWR06
+L power:VCC #PWR025
 U 1 1 60431C5B
 P 2100 4800
-F 0 "#PWR06" H 2100 4650 50  0001 C CNN
+F 0 "#PWR025" H 2100 4650 50  0001 C CNN
 F 1 "VCC" H 2115 4973 50  0000 C CNN
 F 2 "" H 2100 4800 50  0001 C CNN
@@
 	2100 4800 2100 5000
 $Comp
-L Device:R_Small_US R5
+L Device:R_Small_US R7
 U 1 1 60431C63
 P 2200 5150
-F 0 "R5" H 2268 5150 50  0000 L CNN
+F 0 "R7" H 2268 5150 50  0000 L CNN
 F 1 "1" H 2268 5105 50  0001 L CNN
 F 2 "Resistor_SMD:R_0603_1608Metric_Pad0.98x0.95mm_HandSolder" H 2200 5150 50  0001 C CNN
@@
 $EndComp
 $Comp
-L Device:R_Small_US R7
+L Device:R_Small_US R9
 U 1 1 60431C69
 P 2450 5250
-F 0 "R7" H 2518 5250 50  0000 L CNN
+F 0 "R9" H 2518 5250 50  0000 L CNN
 F 1 "1" H 2518 5205 50  0001 L CNN
 F 2 "Resistor_SMD:R_0603_1608Metric_Pad0.98x0.95mm_HandSolder" H 2450 5250 50  0001 C CNN
@@
 $EndComp
 $Comp
-L Device:R_Small_US R9
+L Device:R_Small_US R11
 U 1 1 60431C6F
 P 2600 5650
-F 0 "R9" H 2668 5650 50  0000 L CNN
+F 0 "R11" H 2668 5650 50  0000 L CNN
 F 1 "1" H 2668 5605 50  0001 L CNN
 F 2 "Resistor_SMD:R_0603_1608Metric_Pad0.98x0.95mm_HandSolder" H 2600 5650 50  0001 C CNN
@@
 $EndComp
 $Comp
-L Device:R_Small_US R11
+L Device:R_Small_US R13
 U 1 1 60431C75
 P 2800 5650
-F 0 "R11" H 2868 5650 50  0000 L CNN
+F 0 "R13" H 2868 5650 50  0000 L CNN
 F 1 "1" H 2868 5605 50  0001 L CNN
 F 2 "Resistor_SMD:R_0603_1608Metric_Pad0.98x0.95mm_HandSolder" H 2800 5650 50  0001 C CNN
@@
 Connection ~ 2600 5900
 $Comp
-L power:GND #PWR09
+L power:GND #PWR028
 U 1 1 60431C97
 P 2650 6850
-F 0 "#PWR09" H 2650 6600 50  0001 C CNN
+F 0 "#PWR028" H 2650 6600 50  0001 C CNN
 F 1 "GND" H 2655 6677 50  0000 C CNN
 F 2 "" H 2650 6850 50  0001 C CNN
@@
 	2650 6700 2650 6850
 $Comp
-L power:VCC #PWR010
+L power:VCC #PWR029
 U 1 1 60443477
 P 6700 1350
-F 0 "#PWR010" H 6700 1200 50  0001 C CNN
+F 0 "#PWR029" H 6700 1200 50  0001 C CNN
 F 1 "VCC" H 6715 1523 50  0000 C CNN
 F 2 "" H 6700 1350 50  0001 C CNN
@@
 	6700 1350 6700 1550
 $Comp
-L Device:R_Small_US R12
+L Device:R_Small_US R14
 U 1 1 6044347F
 P 6800 1700
-F 0 "R12" H 6868 1700 50  0000 L CNN
+F 0 "R14" H 6868 1700 50  0000 L CNN
 F 1 "1" H 6868 1655 50  0001 L CNN
 F 2 "Resistor_SMD:R_0603_1608Metric_Pad0.98x0.95mm_HandSolder" H 6800 1700 50  0001 C CNN
@@
 $EndComp
 $Comp
-L Device:R_Small_US R13
+L Device:R_Small_US R15
 U 1 1 60443485
 P 7050 1800
-F 0 "R13" H 7118 1800 50  0000 L CNN
+F 0 "R15" H 7118 1800 50  0000 L CNN
 F 1 "1" H 7118 1755 50  0001 L CNN
 F 2 "Resistor_SMD:R_0603_1608Metric_Pad0.98x0.95mm_HandSolder" H 7050 1800 50  0001 C CNN
@@
 $EndComp
 $Comp
-L Device:R_Small_US R14
+L Device:R_Small_US R16
 U 1 1 6044348B
 P 7200 2200
-F 0 "R14" H 7268 2200 50  0000 L CNN
+F 0 "R16" H 7268 2200 50  0000 L CNN
 F 1 "1" H 7268 2155 50  0001 L CNN
 F 2 "Resistor_SMD:R_0603_1608Metric_Pad0.98x0.95mm_HandSolder" H 7200 2200 50  0001 C CNN
@@
 $EndComp
 $Comp
-L Device:R_Small_US R15
+L Device:R_Small_US R17
 U 1 1 60443491
 P 7400 2200
-F 0 "R15" H 7468 2200 50  0000 L CNN
+F 0 "R17" H 7468 2200 50  0000 L CNN
 F 1 "1" H 7468 2155 50  0001 L CNN
 F 2 "Resistor_SMD:R_0603_1608Metric_Pad0.98x0.95mm_HandSolder" H 7400 2200 50  0001 C CNN
@@
 Connection ~ 7200 2450
 $Comp
-L power:GND #PWR012
+L power:GND #PWR031
 U 1 1 604434B3
 P 7250 3400
-F 0 "#PWR012" H 7250 3150 50  0001 C CNN
+F 0 "#PWR031" H 7250 3150 50  0001 C CNN
 F 1 "GND" H 7255 3227 50  0000 C CNN
 F 2 "" H 7250 3400 50  0001 C CNN
@@
 Connection ~ 2650 3250
 $Comp
-L power:VCC #PWR05
+L power:VCC #PWR024
 U 1 1 6047FB32
 P 2100 2750
-F 0 "#PWR05" H 2100 2600 50  0001 C CNN
+F 0 "#PWR024" H 2100 2600 50  0001 C CNN
 F 1 "VCC" H 2115 2923 50  0000 C CNN
 F 2 "" H 2100 2750 50  0001 C CNN
@@
 $EndComp
 $Comp
-L power:VCC #PWR011
+L power:VCC #PWR030
 U 1 1 6048F78C
 P 6750 2700
-F 0 "#PWR011" H 6750 2550 50  0001 C CNN
+F 0 "#PWR030" H 6750 2550 50  0001 C CNN
 F 1 "VCC" H 6765 2873 50  0000 C CNN
 F 2 "" H 6750 2700 50  0001 C CNN
@@
 $EndComp
 $Comp
-L power:VCC #PWR07
+L power:VCC #PWR026
 U 1 1 6049F67C
 P 2100 6150
-F 0 "#PWR07" H 2100 6000 50  0001 C CNN
+F 0 "#PWR026" H 2100 6000 50  0001 C CNN
 F 1 "VCC" H 2115 6323 50  0000 C CNN
 F 2 "" H 2100 6150 50  0001 C CNN

Commit message: new part placements.
Connections:
- net Motor2/DECAY: now also U5.13 (P10)
- net Motor2/DIR: now also U5.17 (P14); no longer U5.15 (P12)
- net Motor2/ENABLE: now also U5.18 (P15); no longer U5.16 (P13)
- net Motor2/M0: now also U5.16 (P13); no longer U5.14 (P11)
- net Motor2/M1: now also U5.15 (P12); no longer U5.13 (P10)
- net Motor2/TRQ: now also U5.14 (P11)
- net Motor2/~FAULT: now also U5.20 (P17); no longer U5.18 (P15)
- net Motor2/~SLEEP: now also U5.19 (P16); no longer U5.17 (P14)
- net Motor4/DECAY: now also U6.13 (P10)
- net Motor4/DIR: now also U6.17 (P14); no longer U6.15 (P12)
- net Motor4/ENABLE: now also U6.18 (P15); no longer U6.16 (P13)
- net Motor4/M0: now also U6.16 (P13); no longer U6.14 (P11)
- net Motor4/M1: now also U6.15 (P12); no longer U6.13 (P10)
- net Motor4/TRQ: now also U6.14 (P11)
- net Motor4/~FAULT: now also U6.20 (P17); no longer U6.18 (P15)
- net Motor4/~SLEEP: now also U6.19 (P16); no longer U6.17 (P14)
- net Motor6/DECAY: now also U7.13 (P10)
- net Motor6/DIR: now also U7.17 (P14); no longer U7.15 (P12)
- net Motor6/ENABLE: now also U7.18 (P15); no longer U7.16 (P13)
- net Motor6/M0: now also U7.16 (P13); no longer U7.14 (P11)
- net Motor6/M1: now also U7.15 (P12); no longer U7.13 (P10)
- net Motor6/TRQ: now also U7.14 (P11)
- net Motor6/~FAULT: now also U7.20 (P17); no longer U7.18 (P15)
- net Motor6/~SLEEP: now also U7.19 (P16); no longer U7.17 (P14)
Changed lines of the file:
@@
 $EndDescr
 $Sheet
-S 4650 6050 850  1200
+S 4650 6000 850  1200
 U 6036596C
 F0 "Motor4" 50
 F1 "single_driver.sch" 50
-F2 "RRef" I L 4650 7150 50
-F3 "DECAY" I L 4650 6200 50
-F4 "TRQ" I L 4650 6300 50
-F5 "M1" I L 4650 6400 50
-F6 "M0" I L 4650 6500 50
-F7 "DIR" I L 4650 6600 50
-F8 "STEP" I L 4650 7050 50
-F9 "ENABLE" I L 4650 6700 50
-F10 "~SLEEP" I L 4650 6800 50
-F11 "A1" O R 5500 6400 50
-F12 "A2" O R 5500 6500 50
-F13 "B2" O R 5500 6700 50
-F14 "B1" O R 5500 6800 50
-F15 "~FAULT" I L 4650 6900 50
+F2 "RRef" I L 4650 7100 50
+F3 "DECAY" I L 4650 6150 50
+F4 "TRQ" I L 4650 6250 50
+F5 "M1" I L 4650 6350 50
+F6 "M0" I L 4650 6450 50
+F7 "DIR" I L 4650 6550 50
+F8 "STEP" I L 4650 7000 50
+F9 "ENABLE" I L 4650 6650 50
+F10 "~SLEEP" I L 4650 6750 50
+F11 "A1" O R 5500 6350 50
+F12 "A2" O R 5500 6450 50
+F13 "B2" O R 5500 6650 50
+F14 "B1" O R 5500 6750 50
+F15 "~FAULT" I L 4650 6850 50
 $EndSheet
 $Comp
@@
 $EndSheet
 Wire Wire Line
-	3800 2350 4350 2350
-Wire Wire Line
-	4300 2800 4650 2800
-Wire Wire Line
-	3800 2550 4250 2550
-Wire Wire Line
-	4250 2550 4250 2900
-Wire Wire Line
-	4250 2900 4650 2900
-Wire Wire Line
-	3800 2650 4200 2650
-Wire Wire Line
-	4200 2650 4200 3000
-Wire Wire Line
-	4200 3000 4650 3000
-Wire Wire Line
-	3800 2750 4150 2750
-Wire Wire Line
-	4150 2750 4150 3100
-Wire Wire Line
-	4150 3100 4650 3100
-Wire Wire Line
-	3800 2850 4100 2850
-Wire Wire Line
-	4100 2850 4100 3200
-Wire Wire Line
-	4100 3200 4650 3200
-Wire Wire Line
-	3800 2950 4050 2950
-Wire Wire Line
-	4050 2950 4050 3300
-Wire Wire Line
-	4050 3300 4650 3300
-Wire Wire Line
-	3800 3050 4000 3050
-Wire Wire Line
-	4000 3050 4000 3400
-Wire Wire Line
-	4000 3400 4650 3400
-Wire Wire Line
-	4350 2700 4650 2700
-Wire Wire Line
-	4350 2350 4350 2700
-Wire Wire Line
-	4300 2450 4300 2800
-Wire Wire Line
-	3800 2450 4300 2450
-Wire Wire Line
 	3850 1250 4650 1250
 Wire Wire Line
@@
 	4200 5450 4650 5450
 Wire Wire Line
-	3800 5800 4350 5800
-Wire Wire Line
-	4350 5800 4350 6200
-Wire Wire Line
-	4350 6200 4650 6200
-Wire Wire Line
-	3800 5900 4300 5900
-Wire Wire Line
-	4300 5900 4300 6300
-Wire Wire Line
-	4300 6300 4650 6300
-Wire Wire Line
-	3800 6000 4250 6000
-Wire Wire Line
-	4250 6000 4250 6400
-Wire Wire Line
-	4250 6400 4650 6400
-Wire Wire Line
-	4200 6100 4200 6500
-Wire Wire Line
-	4200 6500 4650 6500
-Wire Wire Line
-	3800 6100 4200 6100
-Wire Wire Line
-	3800 6200 4150 6200
-Wire Wire Line
-	4150 6200 4150 6600
-Wire Wire Line
-	4150 6600 4650 6600
-Wire Wire Line
-	3800 6300 4100 6300
-Wire Wire Line
-	4100 6300 4100 6700
-Wire Wire Line
-	4100 6700 4650 6700
-Wire Wire Line
-	3800 6400 4050 6400
-Wire Wire Line
-	4050 6400 4050 6800
-Wire Wire Line
-	4050 6800 4650 6800
-Wire Wire Line
-	3800 6500 4000 6500
-Wire Wire Line
-	4000 6500 4000 6900
-Wire Wire Line
-	4000 6900 4650 6900
-Wire Wire Line
 	4550 5600 4650 5600
 Wire Wire Line
 	4550 5700 4650 5700
 Wire Wire Line
-	4550 7050 4650 7050
-Wire Wire Line
-	4550 7150 4650 7150
+	4550 7000 4650 7000
+Wire Wire Line
+	4550 7100 4650 7100
 Text HLabel 4550 2100 0    50   Input ~ 0
 STEP1
@@
 Text HLabel 4550 5700 0    50   Input ~ 0
 RRef3
-Text HLabel 4550 7050 0    50   Input ~ 0
+Text HLabel 4550 7000 0    50   Input ~ 0
 STEP4
-Text HLabel 4550 7150 0    50   Input ~ 0
+Text HLabel 4550 7100 0    50   Input ~ 0
 RRef4
 $Comp
@@
 Wire Wire Line
 	9200 3550 9300 3550
-Wire Wire Line
-	8650 3400 9300 3400
-Wire Wire Line
-	8650 3050 8650 3400
-Wire Wire Line
-	8400 3050 8650 3050
-Wire Wire Line
-	8700 3300 9300 3300
-Wire Wire Line
-	8700 2950 8700 3300
-Wire Wire Line
-	8400 2950 8700 2950
-Wire Wire Line
-	8750 3200 9300 3200
-Wire Wire Line
-	8750 2850 8750 3200
-Wire Wire Line
-	8400 2850 8750 2850
-Wire Wire Line
-	8800 3100 9300 3100
-Wire Wire Line
-	8800 2750 8800 3100
-Wire Wire Line
-	8400 2750 8800 2750
-Wire Wire Line
-	8850 3000 9300 3000
-Wire Wire Line
-	8850 2650 8850 3000
-Wire Wire Line
-	8400 2650 8850 2650
-Wire Wire Line
-	8900 2900 9300 2900
-Wire Wire Line
-	8900 2550 8900 2900
-Wire Wire Line
-	8400 2550 8900 2550
-Wire Wire Line
-	8950 2800 9300 2800
-Wire Wire Line
-	8950 2450 8950 2800
-Wire Wire Line
-	8400 2450 8950 2450
-Wire Wire Line
-	9000 2700 9300 2700
-Wire Wire Line
-	9000 2350 9000 2700
-Wire Wire Line
-	8400 2350 9000 2350
 Wire Wire Line
 	9200 2200 9300 2200
@@
 Text HLabel 5650 5350 2    50   Output ~ 0
 MOTOR3_B1
-Text HLabel 5650 6400 2    50   Output ~ 0
+Text HLabel 5650 6350 2    50   Output ~ 0
 MOTOR4_A1
-Text HLabel 5650 6500 2    50   Output ~ 0
+Text HLabel 5650 6450 2    50   Output ~ 0
 MOTOR4_A2
-Text HLabel 5650 6700 2    50   Output ~ 0
+Text HLabel 5650 6650 2    50   Output ~ 0
 MOTOR4_B2
-Text HLabel 5650 6800 2    50   Output ~ 0
+Text HLabel 5650 6750 2    50   Output ~ 0
 MOTOR4_B1
 Text HLabel 10300 1450 2    50   Output ~ 0
@@
 	5500 5350 5650 5350
 Wire Wire Line
-	5500 6400 5650 6400
-Wire Wire Line
-	5500 6500 5650 6500
-Wire Wire Line
-	5500 6700 5650 6700
-Wire Wire Line
-	5500 6800 5650 6800
+	5500 6350 5650 6350
+Wire Wire Line
+	5500 6450 5650 6450
+Wire Wire Line
+	5500 6650 5650 6650
+Wire Wire Line
+	5500 6750 5650 6750
+Wire Wire Line
+	3800 2550 4500 2550
+Wire Wire Line
+	4500 2550 4500 2700
+Wire Wire Line
+	4500 2700 4650 2700
+Wire Wire Line
+	3800 2650 4450 2650
+Wire Wire Line
+	4450 2650 4450 2800
+Wire Wire Line
+	4450 2800 4650 2800
+Wire Wire Line
+	4400 2750 4400 2900
+Wire Wire Line
+	4400 2900 4650 2900
+Wire Wire Line
+	3800 2750 4400 2750
+Wire Wire Line
+	3800 2850 4350 2850
+Wire Wire Line
+	4350 2850 4350 3000
+Wire Wire Line
+	4350 3000 4650 3000
+Wire Wire Line
+	3800 2950 4300 2950
+Wire Wire Line
+	4300 2950 4300 3100
+Wire Wire Line
+	4300 3100 4650 3100
+Wire Wire Line
+	3800 3050 4250 3050
+Wire Wire Line
+	4250 3050 4250 3200
+Wire Wire Line
+	4250 3200 4650 3200
+Wire Wire Line
+	3800 3150 4200 3150
+Wire Wire Line
+	4200 3150 4200 3300
+Wire Wire Line
+	4200 3300 4650 3300
+Wire Wire Line
+	3800 3250 4150 3250
+Wire Wire Line
+	4150 3250 4150 3400
+Wire Wire Line
+	4150 3400 4650 3400
+Wire Wire Line
+	3800 6000 4500 6000
+Wire Wire Line
+	4500 6000 4500 6150
+Wire Wire Line
+	4500 6150 4650 6150
+Wire Wire Line
+	3800 6100 4450 6100
+Wire Wire Line
+	4450 6100 4450 6250
+Wire Wire Line
+	4450 6250 4650 6250
+Wire Wire Line
+	4400 6200 4400 6350
+Wire Wire Line
+	4400 6350 4650 6350
+Wire Wire Line
+	3800 6200 4400 6200
+Wire Wire Line
+	3800 6300 4350 6300
+Wire Wire Line
+	4350 6300 4350 6450
+Wire Wire Line
+	4350 6450 4650 6450
+Wire Wire Line
+	3800 6400 4300 6400
+Wire Wire Line
+	4300 6400 4300 6550
+Wire Wire Line
+	4300 6550 4650 6550
+Wire Wire Line
+	3800 6500 4250 6500
+Wire Wire Line
+	4250 6500 4250 6650
+Wire Wire Line
+	4250 6650 4650 6650
+Wire Wire Line
+	3800 6600 4200 6600
+Wire Wire Line
+	4200 6600 4200 6750
+Wire Wire Line
+	4200 6750 4650 6750
+Wire Wire Line
+	3800 6700 4150 6700
+Wire Wire Line
+	4150 6700 4150 6850
+Wire Wire Line
+	4150 6850 4650 6850
+Wire Wire Line
+	8400 2550 9100 2550
+Wire Wire Line
+	9100 2550 9100 2700
+Wire Wire Line
+	8400 2650 9050 2650
+Wire Wire Line
+	9050 2650 9050 2800
+Wire Wire Line
+	9000 2750 9000 2900
+Wire Wire Line
+	8400 2750 9000 2750
+Wire Wire Line
+	8400 2850 8950 2850
+Wire Wire Line
+	8950 2850 8950 3000
+Wire Wire Line
+	8400 2950 8900 2950
+Wire Wire Line
+	8900 2950 8900 3100
+Wire Wire Line
+	8400 3050 8850 3050
+Wire Wire Line
+	8850 3050 8850 3200
+Wire Wire Line
+	8400 3150 8800 3150
+Wire Wire Line
+	8800 3150 8800 3300
+Wire Wire Line
+	8400 3250 8750 3250
+Wire Wire Line
+	8750 3250 8750 3400
+Wire Wire Line
+	9100 2700 9300 2700
+Wire Wire Line
+	9050 2800 9300 2800
+Wire Wire Line
+	9000 2900 9300 2900
+Wire Wire Line
+	8950 3000 9300 3000
+Wire Wire Line
+	8900 3100 9300 3100
+Wire Wire Line
+	8850 3200 9300 3200
+Wire Wire Line
+	8800 3300 9300 3300
+Wire Wire Line
+	8750 3400 9300 3400
 $EndSCHEMATC
