File: robarm_pcb/motor_driver/motor_driver_prj/extConnectors.sch (KiCad schematic (older format))
At the start: 0 parts

Commit message: save
Parts:
- added J1: ZF5S-40-01-T-WT, motor_driver:FPC_40, symbol Connector_Generic:Conn_02x20_Odd_Even
- added J10, J9: Conn_01x01_Male, TestPoint:TestPoint_Pad_4.0x4.0mm, symbol Connector:Conn_01x01_Male
- added J2: Conn_01x04_Male, Connector:FanPinHeader_1x04_P2.54mm_Vertical, symbol Connector:Conn_01x04_Male
- added Q1: BSS138, Package_TO_SOT_SMD:SOT-23, symbol Transistor_FET:BSS138
- added R4, R5: 10k, Resistor_SMD:R_0603_1608Metric_Pad0.98x0.95mm_HandSolder, symbol Device:R_Small_US
Connections:
- net labels added: +12V, +3.3V, +5V, +BATT, FAN_PWM, GND, I2C_SCL, I2C_SDA, ~INT1, ~INT2, ~INT3, ~RESET1, ~RESET2, ~RESET3
- wire segments 24 -> 67
- no-connect marks 0 -> 1
Other:
- note added: "FAN PWM level shift and connector"
- note added: "FPC Connector to RPI"
- note added: "Power Connectors"

Commit message: new part placements.
Connections:
- net labels added: VCC
- net labels removed: +3.3V
Other:
- moved on the sheet: J1, J2, Q1, R4, R5

Commit message: Motor Driver PCB rev 1
Motor Driver PCB rev 1
Parts:
- added H1, H2, H3, H4: MountingHole, MountingHole:MountingHole_3.2mm_M3_ISO14580, symbol Mechanical:MountingHole
Connections:
- net GND: now also J1.1 (Pin_1), J1.10 (Pin_10), J1.12 (Pin_12), J1.15 (Pin_15), J1.16 (Pin_16), J1.17 (Pin_17), J1.18 (Pin_18), J1.2 (Pin_2), J1.22 (Pin_22), J1.23 (Pin_23), J1.24 (Pin_24), J1.26 (Pin_26), J1.27 (Pin_27), J1.28 (Pin_28), J1.32 (Pin_32), J1.33 (Pin_33), J1.35 (Pin_35), J1.36 (Pin_36), J1.37 (Pin_37), J1.38 (Pin_38), J1.4 (Pin_4), J1.40 (Pin_40), J1.7 (Pin_7), J1.8 (Pin_8)
Other:
- note added: "Mounting Holes"
Changed lines of the file:
@@
 	3250 2750 3000 2750
 Wire Wire Line
-	3000 1950 3000 2750
+	3000 1950 3000 2250
 Connection ~ 3000 2750
 Wire Wire Line
-	3000 2750 3000 3450
+	3000 2750 3000 2850
 $Comp
 L power:GND #PWR022
@@
 	3750 1750 3950 1750
 Wire Wire Line
-	3950 1750 3950 2150
+	3950 1750 3950 1850
 Wire Wire Line
 	3750 2150 3950 2150
 Connection ~ 3950 2150
 Wire Wire Line
-	3950 2150 3950 2450
+	3950 2150 3950 2250
 Wire Wire Line
 	3750 2450 3950 2450
 Connection ~ 3950 2450
 Wire Wire Line
-	3950 2450 3950 2950
+	3950 2450 3950 2550
 Wire Wire Line
 	3750 2950 3950 2950
 Connection ~ 3950 2950
 Wire Wire Line
-	3950 2950 3950 3150
+	3950 2950 3950 3050
 Wire Wire Line
 	3750 3150 3950 3150
 Connection ~ 3950 3150
 Wire Wire Line
-	3950 3150 3950 3700
+	3950 3150 3950 3250
 Text HLabel 2850 1650 0    50   Input ~ 0
 I2C_SDA
@@
 	1    0    0    -1
 $EndComp
+Wire Wire Line
+	3250 1550 3000 1550
+Wire Wire Line
+	3000 1550 3000 1850
+Connection ~ 3000 1950
+Wire Wire Line
+	3250 1850 3000 1850
+Connection ~ 3000 1850
+Wire Wire Line
+	3000 1850 3000 1950
+Wire Wire Line
+	3250 2250 3000 2250
+Connection ~ 3000 2250
+Wire Wire Line
+	3000 2250 3000 2350
+Wire Wire Line
+	3250 2350 3000 2350
+Connection ~ 3000 2350
+Wire Wire Line
+	3000 2350 3000 2650
+Wire Wire Line
+	3250 2650 3000 2650
+Connection ~ 3000 2650
+Wire Wire Line
+	3000 2650 3000 2750
+Wire Wire Line
+	3250 2850 3000 2850
+Connection ~ 3000 2850
+Wire Wire Line
+	3000 2850 3000 3150
+Wire Wire Line
+	3250 3150 3000 3150
+Connection ~ 3000 3150
+Wire Wire Line
+	3000 3150 3000 3250
+Wire Wire Line
+	3250 3250 3000 3250
+Connection ~ 3000 3250
+Wire Wire Line
+	3000 3250 3000 3350
+Wire Wire Line
+	3250 3350 3000 3350
+Connection ~ 3000 3350
+Wire Wire Line
+	3000 3350 3000 3450
+Wire Wire Line
+	3750 3450 3950 3450
+Connection ~ 3950 3450
+Wire Wire Line
+	3950 3450 3950 3700
+Wire Wire Line
+	3750 3350 3950 3350
+Connection ~ 3950 3350
+Wire Wire Line
+	3950 3350 3950 3450
+Wire Wire Line
+	3750 3250 3950 3250
+Connection ~ 3950 3250
+Wire Wire Line
+	3950 3250 3950 3350
+Wire Wire Line
+	3750 3050 3950 3050
+Connection ~ 3950 3050
+Wire Wire Line
+	3950 3050 3950 3150
+Wire Wire Line
+	3750 2850 3950 2850
+Connection ~ 3950 2850
+Wire Wire Line
+	3950 2850 3950 2950
+Wire Wire Line
+	3750 2750 3950 2750
+Connection ~ 3950 2750
+Wire Wire Line
+	3950 2750 3950 2850
+Wire Wire Line
+	3750 2650 3950 2650
+Connection ~ 3950 2650
+Wire Wire Line
+	3950 2650 3950 2750
+Wire Wire Line
+	3750 2550 3950 2550
+Connection ~ 3950 2550
+Wire Wire Line
+	3950 2550 3950 2650
+Wire Wire Line
+	3750 2350 3950 2350
+Connection ~ 3950 2350
+Wire Wire Line
+	3950 2350 3950 2450
+Wire Wire Line
+	3750 2250 3950 2250
+Connection ~ 3950 2250
+Wire Wire Line
+	3950 2250 3950 2350
+Wire Wire Line
+	3750 2050 3950 2050
+Connection ~ 3950 2050
+Wire Wire Line
+	3950 2050 3950 2150
+Wire Wire Line
+	3750 1950 3950 1950
+Connection ~ 3950 1950
+Wire Wire Line
+	3950 1950 3950 2050
+Wire Wire Line
+	3750 1850 3950 1850
+Connection ~ 3950 1850
+Wire Wire Line
+	3950 1850 3950 1950
+Wire Wire Line
+	3750 1650 3950 1650
+Wire Wire Line
+	3950 1650 3950 1750
+Connection ~ 3950 1750
+Wire Wire Line
+	3750 1550 3950 1550
+Wire Wire Line
+	3950 1550 3950 1650
+Connection ~ 3950 1650
+$Comp
+L Mechanical:MountingHole H1
+U 1 1 6092C97D
+P 5900 5050
+F 0 "H1" H 6000 5096 50  0000 L CNN
+F 1 "MountingHole" H 6000 5005 50  0000 L CNN
+F 2 "MountingHole:MountingHole_3.2mm_M3_ISO14580" H 5900 5050 50  0001 C CNN
+F 3 "~" H 5900 5050 50  0001 C CNN
+	1    5900 5050
+	1    0    0    -1
+$EndComp
+$Comp
+L Mechanical:MountingHole H2
+U 1 1 6092D5B7
+P 5900 5350
+F 0 "H2" H 6000 5396 50  0000 L CNN
+F 1 "MountingHole" H 6000 5305 50  0000 L CNN
+F 2 "MountingHole:MountingHole_3.2mm_M3_ISO14580" H 5900 5350 50  0001 C CNN
+F 3 "~" H 5900 5350 50  0001 C CNN
+	1    5900 5350
+	1    0    0    -1
+$EndComp
+$Comp
+L Mechanical:MountingHole H3
+U 1 1 6092DCE4
+P 5900 5650
+F 0 "H3" H 6000 5696 50  0000 L CNN
+F 1 "MountingHole" H 6000 5605 50  0000 L CNN
+F 2 "MountingHole:MountingHole_3.2mm_M3_ISO14580" H 5900 5650 50  0001 C CNN
+F 3 "~" H 5900 5650 50  0001 C CNN
+	1    5900 5650
+	1    0    0    -1
+$EndComp
+$Comp
+L Mechanical:MountingHole H4
+U 1 1 6092EF37
+P 5900 5950
+F 0 "H4" H 6000 5996 50  0000 L CNN
+F 1 "MountingHole" H 6000 5905 50  0000 L CNN
+F 2 "MountingHole:MountingHole_3.2mm_M3_ISO14580" H 5900 5950 50  0001 C CNN
+F 3 "~" H 5900 5950 50  0001 C CNN
+	1    5900 5950
+	1    0    0    -1
+$EndComp
+Wire Notes Line
+	5550 6300 6750 6300
+Wire Notes Line
+	6750 6300 6750 4500
+Wire Notes Line
+	6750 4500 5550 4500
+Wire Notes Line
+	5550 4500 5550 6300
+Text Notes 5800 4700 0    50   ~ 0
+Mounting Holes
 $EndSCHEMATC
