File: robarm_pcb/motor_driver/motor_driver_prj/motor_driver_prj.kicad_pcb (KiCad board)
At the start: 2 copper layers, 114.3 x 76.2 mm, 82 parts, among them U1 TCA9539PWR, U10 DRV8886PWPR‎, U2 TCA9539PWR, U3 TCA9539PWR, U4 PCA9685PW, U5 DRV8886PWPR‎, U6 DRV8886PWPR‎, U7 DRV8886PWPR‎, U8 DRV8886PWPR‎, U9 DRV8886PWPR‎

Commit message: save
Parts:
- added C49: 0.47uF, Capacitor_SMD:C_0805_2012Metric_Pad1.18x1.45mm_HandSolder, F.Cu at (178.4, 125.7)
- added C50: 0.47uF, Capacitor_SMD:C_0805_2012Metric_Pad1.18x1.45mm_HandSolder, F.Cu at (179.3, 123.4)
- added C51: 0.022uF, Capacitor_SMD:C_0603_1608Metric_Pad1.08x0.95mm_HandSolder, F.Cu at (183.9, 123.1)
- added C52: 0.01uF, Capacitor_SMD:C_0603_1608Metric_Pad1.08x0.95mm_HandSolder, F.Cu at (180.7, 126.1)
- added C53: 0.22uF, Capacitor_SMD:C_0603_1608Metric_Pad1.08x0.95mm_HandSolder, F.Cu at (189.3, 116.3)
- added C54: 100uF, Capacitor_SMD:CP_Elec_8x6.2, F.Cu at (164.5, 106.7)
- added C55: 0.01uF, Capacitor_SMD:C_0603_1608Metric_Pad1.08x0.95mm_HandSolder, F.Cu at (189.3, 118.8)
- added D1: B340-13-F, footprints:B340-13-F, F.Cu at (116.8, 137.2)
- added D2: B340-13-F, footprints:B340-13-F, F.Cu at (155.6, 137.2)
- added J1: ZF5S-40-01-T-WT, motor_driver:FPC_40, F.Cu at (104.1, 102.9)
- added J10: Conn_01x01_Male, TestPoint:TestPoint_Pad_4.0x4.0mm, F.Cu at (104.1, 124.5)
- added J2: Conn_01x04_Male, Connector:FanPinHeader_1x04_P2.54mm_Vertical, F.Cu at (134.6, 112.4)
- added J3: Conn_01x04_Male, Connector_Phoenix_MSTB:PhoenixContact_MSTBVA_2,5_4-G-5,08_1x04_P5.08mm_Vertical, F.Cu at (126.4, 64.1)
- added J4: Conn_01x04_Male, Connector_Phoenix_MSTB:PhoenixContact_MSTBVA_2,5_4-G-5,08_1x04_P5.08mm_Vertical, F.Cu at (149.9, 64.1)
- added J5: Conn_01x04_Male, Connector_Phoenix_MSTB:PhoenixContact_MSTBVA_2,5_4-G-5,08_1x04_P5.08mm_Vertical, F.Cu at (173.4, 64.1)
- added J6: Conn_01x04_Male, Connector_Phoenix_MSTB:PhoenixContact_MSTBVA_2,5_4-G-5,08_1x04_P5.08mm_Vertical, F.Cu at (196.8, 64.1)
- added J7: Conn_01x04_Male, Connector_Phoenix_MSTB:PhoenixContact_MSTBVA_2,5_4-G-5,08_1x04_P5.08mm_Vertical, F.Cu at (207.0, 115.6)
- added J8: Conn_01x04_Male, Connector_Phoenix_MSTB:PhoenixContact_MSTBVA_2,5_4-G-5,08_1x04_P5.08mm_Vertical, F.Cu at (207.0, 139.1)
- added J9: Conn_01x01_Male, TestPoint:TestPoint_Pad_4.0x4.0mm, F.Cu at (104.1, 134.6)
- added L1: 100uH, motor_driver:SRR1280A-101M, F.Cu at (127.0, 135.9)
- added L2: 100uH, motor_driver:SRR1280A-101M, F.Cu at (165.7, 135.9)
- added Q1: BSS138, Package_TO_SOT_SMD:SOT-23, F.Cu at (140.3, 118.1)
- added R25: R_Small_US, Resistor_SMD:R_0603_1608Metric_Pad0.98x0.95mm_HandSolder, F.Cu at (160.0, 91.4)
- added R26: R_Small_US, Resistor_SMD:R_0603_1608Metric_Pad0.98x0.95mm_HandSolder, F.Cu at (139.7, 89.5)
- added R27: R_Small_US, Resistor_SMD:R_0603_1608Metric_Pad0.98x0.95mm_HandSolder, F.Cu at (142.9, 92.7)
- added R28: rref, Resistor_SMD:R_0603_1608Metric_Pad0.98x0.95mm_HandSolder, F.Cu at (139.1, 92.7)
- added R29: R_Small_US, Resistor_SMD:R_0603_1608Metric_Pad0.98x0.95mm_HandSolder, F.Cu at (137.2, 92.7)
- added R30: R_Small_US, Resistor_SMD:R_0603_1608Metric_Pad0.98x0.95mm_HandSolder, F.Cu at (121.3, 91.4)
- added R31: R_Small_US, Resistor_SMD:R_0603_1608Metric_Pad0.98x0.95mm_HandSolder, F.Cu at (119.4, 91.4)
- added R32: rref, Resistor_SMD:R_0603_1608Metric_Pad0.98x0.95mm_HandSolder, F.Cu at (115.6, 91.4)
- added R33: R_Small_US, Resistor_SMD:R_0603_1608Metric_Pad0.98x0.95mm_HandSolder, F.Cu at (113.7, 91.4)
- added R34: R_Small_US, Resistor_SMD:R_0603_1608Metric_Pad0.98x0.95mm_HandSolder, F.Cu at (195.4, 114.7)
- added R35: R_Small_US, Resistor_SMD:R_0603_1608Metric_Pad0.98x0.95mm_HandSolder, F.Cu at (195.4, 119.7)
- added R36: rref, Resistor_SMD:R_0603_1608Metric_Pad0.98x0.95mm_HandSolder, F.Cu at (199.8, 114.7)
- added R37: R_Small_US, Resistor_SMD:R_0603_1608Metric_Pad0.98x0.95mm_HandSolder, F.Cu at (195.4, 117.2)
- added R38: R_Small_US, Resistor_SMD:R_0603_1608Metric_Pad0.98x0.95mm_HandSolder, F.Cu at (191.1, 127.0)
- added R39: R_Small_US, Resistor_SMD:R_0603_1608Metric_Pad0.98x0.95mm_HandSolder, F.Cu at (189.3, 113.8)
- added R40: rref, Resistor_SMD:R_0603_1608Metric_Pad0.98x0.95mm_HandSolder, F.Cu at (173.4, 139.7)
- added R41: R_Small_US, Resistor_SMD:R_0603_1608Metric_Pad0.98x0.95mm_HandSolder, F.Cu at (176.3, 126.1)
- added U11: DRV8886PWPR‎, motor_driver:DRV8886_HTSSOP-24, F.Cu at (115.6, 81.9)
- added U12: DRV8886PWPR‎, motor_driver:DRV8886_HTSSOP-24, F.Cu at (189.9, 95.9)
- added U13: DRV8886PWPR‎, motor_driver:DRV8886_HTSSOP-24, F.Cu at (189.2, 128.3)
- C1: value 0.1uF -> 10uF; footprint Capacitor_SMD:C_0603_1608Metric_Pad1.08x0.95mm_HandSolder -> Capacitor_SMD:C_0805_2012Metric_Pad1.18x1.45mm_HandSolder
- C11, C19, C27, C35, C43: value 0.47uF -> 0.022uF; footprint Capacitor_SMD:C_0805_2012Metric_Pad1.18x1.45mm_HandSolder -> Capacitor_SMD:C_0603_1608Metric_Pad1.08x0.95mm_HandSolder
- C12, C20, C28, C36, C44: value 0.022uF -> 0.01uF
- C13, C21, C29, C37, C45: value 0.01uF -> 0.22uF
- C14, C22, C30, C38, C46: value 0.22uF -> 100uF; footprint Capacitor_SMD:C_0603_1608Metric_Pad1.08x0.95mm_HandSolder -> Capacitor_SMD:CP_Elec_8x6.2
- C15, C23, C31, C39, C47: value 100uF -> 0.01uF; footprint Capacitor_SMD:CP_Elec_8x6.2 -> Capacitor_SMD:C_0603_1608Metric_Pad1.08x0.95mm_HandSolder
- C16, C24, C32, C40, C48, C5, C8: value 0.01uF -> 0.1uF
- C17, C25, C33, C41, C9: value 0.1uF -> 0.47uF; footprint Capacitor_SMD:C_0603_1608Metric_Pad1.08x0.95mm_HandSolder -> Capacitor_SMD:C_0805_2012Metric_Pad1.18x1.45mm_HandSolder
- C2, C3: value 0.47uF -> 100uF; footprint Capacitor_SMD:C_0805_2012Metric_Pad1.18x1.45mm_HandSolder -> Capacitor_SMD:CP_Elec_8x6.2
- C4: value 0.022uF -> 10uF; footprint Capacitor_SMD:C_0603_1608Metric_Pad1.08x0.95mm_HandSolder -> Capacitor_SMD:C_0805_2012Metric_Pad1.18x1.45mm_HandSolder
- C6: value 0.22uF -> 1000uF; footprint Capacitor_SMD:C_0603_1608Metric_Pad1.08x0.95mm_HandSolder -> Capacitor_SMD:CP_Elec_8x6.2
- C7: value 100uF -> 1000uF
- R10, R12, R13, R14, R16, R17, R6, R8, R9: value R_Small_US -> 1
- R11, R15, R7: value rref -> 1
- R19, R23, R3: value rref -> R_Small_US
- R20, R24: value R_Small_US -> rref
- R4, R5: value R_Small_US -> 10k
- U1: value TCA9539PWR -> MC78M05_TO252; footprint motor_driver:TCA9539_TSSOP-24 -> Package_TO_SOT_SMD:TO-252-2
- U2: value TCA9539PWR -> LM2576SX-3.3; footprint motor_driver:TCA9539_TSSOP-24 -> motor_driver:LM2576SX_TO263-5
- U3: value TCA9539PWR -> LM2576S-12; footprint motor_driver:TCA9539_TSSOP-24 -> motor_driver:LM2576SX_TO263-5
- U5, U6, U7: value DRV8886PWPR‎ -> TCA9539PWR; footprint motor_driver:DRV8886_HTSSOP-24 -> motor_driver:TCA9539_TSSOP-24
- moved C2 203.1 mm to (114.3, 124.5), turned to 90 degrees
- moved R4 199.7 mm to (137.2, 118.1), turned to 90 degrees
- moved C1 197.7 mm to (146.1, 129.5), turned to 180 degrees
- moved C4 195.2 mm to (146.1, 119.4), turned to 180 degrees
- moved C33 193.5 mm to (110.5, 89.7), turned to 180 degrees
- moved C6 189.1 mm to (141.0, 135.9)
- moved C5 186.7 mm to (146.1, 117.5), turned to 180 degrees
- moved C24 183.4 mm to (141.0, 92.7), turned to 90 degrees
- moved C3 177.6 mm to (153.0, 124.5), turned to 90 degrees
- moved C32 176.6 mm to (117.5, 91.4), turned to 90 degrees
- moved C39 173.9 mm to (109.9, 75.6), turned to 180 degrees
- moved C35 171.6 mm to (120.0, 75.6), turned to 180 degrees
- moved C34 170.1 mm to (110.5, 87.6), turned to 180 degrees
- moved C38 169.8 mm to (126.4, 75.6), turned to 270 degrees
- moved C37 168.5 mm to (120.0, 73.9), turned to 180 degrees
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Connections:
- C1 pad 1: Net-(C1-Pad1) -> +12V
- C11 pad 2: GND -> Net-(C11-Pad2)
- C12 pad 1: Net-(C12-Pad1) -> +BATT
- C12 pad 2: Net-(C12-Pad2) -> GND
- C13 pad 1: +BATT -> Net-(C13-Pad1)
- C13 pad 2: GND -> +BATT
- C14 pad 1: Net-(C14-Pad1) -> +BATT
- C14 pad 2: +BATT -> GND
- C16 pad 1: +BATT -> Net-(C16-Pad1)
- C19 pad 2: GND -> Net-(C19-Pad2)
- C2 pad 1: Net-(C2-Pad1) -> +BATT
- C20 pad 1: Net-(C20-Pad1) -> +BATT
- C20 pad 2: Net-(C20-Pad2) -> GND
- C21 pad 1: +BATT -> Net-(C21-Pad1)
- C21 pad 2: GND -> +BATT
- C22 pad 1: Net-(C22-Pad1) -> +BATT
- C22 pad 2: +BATT -> GND
- C24 pad 1: +BATT -> Net-(C24-Pad1)
- C27 pad 2: GND -> Net-(C27-Pad2)
- C28 pad 1: Net-(C28-Pad1) -> +BATT
- C28 pad 2: Net-(C28-Pad2) -> GND
- C29 pad 1: +BATT -> Net-(C29-Pad1)
- C29 pad 2: GND -> +BATT
- C3 pad 1: Net-(C3-Pad1) -> +BATT
- C30 pad 1: Net-(C30-Pad1) -> +BATT
- C30 pad 2: +BATT -> GND
- C32 pad 1: +BATT -> Net-(C32-Pad1)
- C35 pad 2: GND -> Net-(C35-Pad2)
- C36 pad 1: Net-(C36-Pad1) -> +BATT
- C36 pad 2: Net-(C36-Pad2) -> GND
- C37 pad 1: +BATT -> Net-(C37-Pad1)
- C37 pad 2: GND -> +BATT
- C38 pad 1: Net-(C38-Pad1) -> +BATT
- C38 pad 2: +BATT -> GND
- C4 pad 1: Net-(C4-Pad1) -> +5V
- C4 pad 2: Net-(C4-Pad2) -> GND
- C40 pad 1: +BATT -> Net-(C40-Pad1)
- C43 pad 2: GND -> Net-(C43-Pad2)
- C44 pad 1: Net-(C44-Pad1) -> +BATT
- C44 pad 2: Net-(C44-Pad2) -> GND
- C45 pad 1: +BATT -> Net-(C45-Pad1)
- C45 pad 2: GND -> +BATT
- C46 pad 1: Net-(C46-Pad1) -> +BATT
- C46 pad 2: +BATT -> GND
- C48 pad 1: +BATT -> Net-(C48-Pad1)
- C5 pad 1: +BATT -> +5V
- C6 pad 1: Net-(C6-Pad1) -> VCC
- C6 pad 2: +BATT -> GND
- C7 pad 1: +BATT -> +12V
- C8 pad 1: +BATT -> Net-(C8-Pad1)
- R1 pad 1: RRef4 -> VCC
- R1 pad 2: Net-(C1-Pad1) -> /I2C_SCL
- R10 pad 1: Net-(C17-Pad1) -> VCC
- R10 pad 2: GND -> /AllDrivers/~RESET1
- R11 pad 1: Net-(C17-Pad1) -> VCC
- R11 pad 2: Net-(R11-Pad2) -> /AllDrivers/~RESET2
- R12 pad 1: /Motor5/~FAULT -> VCC
- R12 pad 2: Net-(C18-Pad1) -> /AllDrivers/~INT1
- R13 pad 1: RRef3 -> VCC
- R13 pad 2: Net-(C25-Pad1) -> /AllDrivers/~INT2
- R14 pad 1: Net-(C25-Pad1) -> VCC
- R14 pad 2: GND -> /I2C_SDA
- R15 pad 1: Net-(C25-Pad1) -> VCC
- R15 pad 2: Net-(R15-Pad2) -> /I2C_SCL
- R16 pad 1: /Motor3/~FAULT -> VCC
- R16 pad 2: Net-(C26-Pad1) -> /AllDrivers/~RESET3
- R17 pad 1: RRef2 -> VCC
- R17 pad 2: Net-(C33-Pad1) -> /AllDrivers/~INT3
- R18 pad 1: Net-(C33-Pad1) -> /AllDrivers/RRef4
- R18 pad 2: GND -> Net-(C8-Pad1)
- R19 pad 1: Net-(C33-Pad1) -> Net-(C8-Pad1)
- R19 pad 2: Net-(R19-Pad2) -> GND
- R2 pad 1: Net-(C1-Pad1) -> VCC
- R2 pad 2: GND -> /I2C_SDA
- R20 pad 1: /Motor2/~FAULT -> Net-(C8-Pad1)
- R20 pad 2: Net-(C34-Pad1) -> Net-(R20-Pad2)
- R21 pad 1: RRef1 -> /AllDrivers/Motor4/~FAULT
- R21 pad 2: Net-(C41-Pad1) -> Net-(C9-Pad1)
- R22 pad 1: Net-(C41-Pad1) -> /AllDrivers/RRef3
- R22 pad 2: GND -> Net-(C16-Pad1)
- R23 pad 1: Net-(C41-Pad1) -> Net-(C16-Pad1)
- R23 pad 2: Net-(R23-Pad2) -> GND
- R24 pad 1: /Motor1/~FAULT -> Net-(C16-Pad1)
- R24 pad 2: Net-(C42-Pad1) -> Net-(R24-Pad2)
- R3 pad 1: Net-(C1-Pad1) -> VCC
- R4 pad 1: /Motor4/~FAULT -> /FAN_PWM
- R4 pad 2: Net-(C2-Pad1) -> +3V3
- R5 pad 1: RRef6 -> +5V
- R5 pad 2: Net-(C9-Pad1) -> Net-(J2-Pad1)
- R6 pad 1: Net-(C9-Pad1) -> VCC
- R6 pad 2: GND -> /I2C_SDA
- R7 pad 1: Net-(C9-Pad1) -> VCC
- R7 pad 2: Net-(R7-Pad2) -> /I2C_SDA
- R8 pad 1: /Motor6/~FAULT -> VCC
- R8 pad 2: Net-(C10-Pad1) -> /I2C_SCL
- R9 pad 1: RRef5 -> VCC
- R9 pad 2: Net-(C17-Pad1) -> /I2C_SCL
- U1 pad 1: Net-(U1-Pad1) -> +12V
- U1 pad 2: Net-(U1-Pad2) -> GND
- U1 pad 3: Net-(U1-Pad3) -> +5V
- U10 pad 1: Net-(C44-Pad1) -> Net-(C27-Pad1)
- U10 pad 10: /Motor1/B1 -> /AllDrivers/MOTOR2_B1
- U10 pad 13: Net-(C43-Pad1) -> Net-(C26-Pad1)
- U10 pad 14: Net-(C42-Pad1) -> Net-(C25-Pad1)
- U10 pad 15: /Motor1/~FAULT -> /AllDrivers/Motor2/~FAULT
- U10 pad 16: Net-(R23-Pad2) -> Net-(R28-Pad2)
- U10 pad 17: /Motor1/~SLEEP -> /AllDrivers/Motor2/~SLEEP
- U10 pad 18: /Motor1/ENABLE -> /AllDrivers/Motor2/ENABLE
- U10 pad 19: STEP1 -> /AllDrivers/STEP2
- U10 pad 2: Net-(C44-Pad2) -> Net-(C27-Pad2)
- U10 pad 20: /Motor1/DIR -> /AllDrivers/Motor2/DIR
- U10 pad 21: /Motor1/M0 -> /AllDrivers/Motor2/M0
- U10 pad 22: /Motor1/M1 -> /AllDrivers/Motor2/M1
- U10 pad 23: /Motor1/TRQ -> /AllDrivers/Motor2/TRQ
- U10 pad 24: /Motor1/DECAY -> (no net)
- U10 pad 3: Net-(C46-Pad1) -> Net-(C29-Pad1)
- U10 pad 5: /Motor1/A1 -> /AllDrivers/MOTOR2_A1
- U10 pad 7: /Motor1/A2 -> /AllDrivers/MOTOR2_A2
- U10 pad 8: /Motor1/B2 -> /AllDrivers/MOTOR2_B2
- U2 pad 1: Net-(U2-Pad1) -> +BATT
- U2 pad 3: Net-(U2-Pad3) -> GND
- U2 pad 4: /Motor3/DECAY -> VCC
- U2 pad 5: /Motor3/TRQ -> GND
- U3 pad 1: Net-(U3-Pad1) -> +BATT
- U3 pad 3: Net-(U3-Pad3) -> GND
- U3 pad 4: /Motor5/DECAY -> +12V
- U3 pad 5: /Motor5/TRQ -> GND
- U4 pad 1: Net-(U4-Pad1) -> GND
- U4 pad 10: Net-(U4-Pad10) -> /AllDrivers/STEP3
- U4 pad 11: Net-(U4-Pad11) -> /AllDrivers/RRef3
- U4 pad 12: Net-(U4-Pad12) -> /AllDrivers/STEP4
- U4 pad 13: Net-(U4-Pad13) -> /AllDrivers/RRef4
- U4 pad 14: Net-(U4-Pad14) -> GND
- U4 pad 15: Net-(U4-Pad15) -> /AllDrivers/RRef5
- U4 pad 16: Net-(U4-Pad16) -> /AllDrivers/STEP5
- U4 pad 17: Net-(U4-Pad17) -> /AllDrivers/RRef6
- U4 pad 18: Net-(U4-Pad18) -> /AllDrivers/STEP6
- U4 pad 19: Net-(U4-Pad19) -> (no net)
- U4 pad 2: Net-(U4-Pad2) -> GND
- U4 pad 20: Net-(U4-Pad20) -> (no net)
- U4 pad 21: Net-(U4-Pad21) -> (no net)
- U4 pad 22: Net-(U4-Pad22) -> /FAN_PWM
- U4 pad 23: Net-(U4-Pad23) -> Net-(R3-Pad2)
- U4 pad 24: Net-(U4-Pad24) -> VCC
- U4 pad 25: Net-(U4-Pad25) -> GND
- U4 pad 26: Net-(U4-Pad26) -> /I2C_SCL
- U4 pad 27: Net-(U4-Pad27) -> /I2C_SDA
- U4 pad 28: Net-(U4-Pad28) -> VCC
- U4 pad 3: Net-(U4-Pad3) -> GND
- U4 pad 4: Net-(U4-Pad4) -> GND
- U4 pad 5: Net-(U4-Pad5) -> GND
- U4 pad 6: Net-(U4-Pad6) -> /AllDrivers/STEP1
- U4 pad 7: Net-(U4-Pad7) -> /AllDrivers/RRef1
- U4 pad 8: Net-(U4-Pad8) -> /AllDrivers/STEP2
- U4 pad 9: Net-(U4-Pad9) -> /AllDrivers/RRef2
- U5 pad 1: Net-(C4-Pad1) -> /AllDrivers/~INT1
- U5 pad 10: /Motor4/B1 -> /AllDrivers/Motor1/~SLEEP
- U5 pad 11: +BATT -> /AllDrivers/Motor1/~FAULT
- U5 pad 13: Net-(C3-Pad1) -> /AllDrivers/Motor2/TRQ
- U5 pad 14: Net-(C2-Pad1) -> /AllDrivers/Motor2/M1
- U5 pad 15: /Motor4/~FAULT -> /AllDrivers/Motor2/M0
- U5 pad 16: Net-(R3-Pad2) -> /AllDrivers/Motor2/DIR
- U5 pad 17: /Motor4/~SLEEP -> /AllDrivers/Motor2/ENABLE
- U5 pad 18: /Motor4/ENABLE -> /AllDrivers/Motor2/~SLEEP
- U5 pad 19: STEP4 -> /AllDrivers/Motor2/~FAULT
- U5 pad 2: Net-(C4-Pad2) -> GND
- U5 pad 20: /Motor4/DIR -> (no net)
- U5 pad 21: /Motor4/M0 -> VCC
- U5 pad 22: /Motor4/M1 -> /I2C_SCL
- U5 pad 23: /Motor4/TRQ -> /I2C_SDA
- U5 pad 24: /Motor4/DECAY -> VCC
- U5 pad 3: Net-(C6-Pad1) -> /AllDrivers/~RESET1
- U5 pad 4: +BATT -> /AllDrivers/Motor1/DECAY
- U5 pad 5: /Motor4/A1 -> /AllDrivers/Motor1/TRQ
- U5 pad 6: GND -> /AllDrivers/Motor1/M1
- U5 pad 7: /Motor4/A2 -> /AllDrivers/Motor1/M0
- U5 pad 8: /Motor4/B2 -> /AllDrivers/Motor1/DIR
- U5 pad 9: GND -> /AllDrivers/Motor1/ENABLE
- U6 pad 1: Net-(C12-Pad1) -> /AllDrivers/~INT2
- U6 pad 10: /Motor6/B1 -> /AllDrivers/Motor3/~SLEEP
- U6 pad 11: +BATT -> /AllDrivers/Motor3/~FAULT
- U6 pad 13: Net-(C11-Pad1) -> /AllDrivers/Motor4/TRQ
- U6 pad 14: Net-(C10-Pad1) -> /AllDrivers/Motor4/M1
- U6 pad 15: /Motor6/~FAULT -> /AllDrivers/Motor4/M0
- U6 pad 16: Net-(R7-Pad2) -> /AllDrivers/Motor4/DIR
- U6 pad 17: /Motor6/~SLEEP -> /AllDrivers/Motor4/ENABLE
- U6 pad 18: /Motor6/ENABLE -> /AllDrivers/Motor4/~SLEEP
- U6 pad 19: STEP6 -> /AllDrivers/Motor4/~FAULT
- U6 pad 2: Net-(C12-Pad2) -> VCC
- U6 pad 20: /Motor6/DIR -> (no net)
- U6 pad 21: /Motor6/M0 -> GND
- U6 pad 22: /Motor6/M1 -> /I2C_SCL
- U6 pad 23: /Motor6/TRQ -> /I2C_SDA
- U6 pad 24: /Motor6/DECAY -> VCC
- U6 pad 3: Net-(C14-Pad1) -> /AllDrivers/~RESET2
- U6 pad 4: +BATT -> /AllDrivers/Motor3/DECAY
- U6 pad 5: /Motor6/A1 -> /AllDrivers/Motor3/TRQ
- U6 pad 6: GND -> /AllDrivers/Motor3/M1
- U6 pad 7: /Motor6/A2 -> /AllDrivers/Motor3/M0
- U6 pad 8: /Motor6/B2 -> /AllDrivers/Motor3/DIR
- U6 pad 9: GND -> /AllDrivers/Motor3/ENABLE
- U7 pad 1: Net-(C20-Pad1) -> /AllDrivers/~INT3
- U7 pad 10: /Motor5/B1 -> /AllDrivers/Motor5/~SLEEP
- U7 pad 11: +BATT -> /AllDrivers/Motor5/~FAULT
- U7 pad 13: Net-(C19-Pad1) -> /AllDrivers/Motor6/TRQ
- U7 pad 14: Net-(C18-Pad1) -> /AllDrivers/Motor6/M1
- U7 pad 15: /Motor5/~FAULT -> /AllDrivers/Motor6/M0
- U7 pad 16: Net-(R11-Pad2) -> /AllDrivers/Motor6/DIR
- U7 pad 17: /Motor5/~SLEEP -> /AllDrivers/Motor6/ENABLE
- U7 pad 18: /Motor5/ENABLE -> /AllDrivers/Motor6/~SLEEP
- U7 pad 19: STEP5 -> /AllDrivers/Motor6/~FAULT
- U7 pad 2: Net-(C20-Pad2) -> VCC
- U7 pad 20: /Motor5/DIR -> (no net)
- U7 pad 21: /Motor5/M0 -> VCC
- U7 pad 22: /Motor5/M1 -> /I2C_SCL
- U7 pad 23: /Motor5/TRQ -> /I2C_SDA
- U7 pad 24: /Motor5/DECAY -> VCC
- U7 pad 3: Net-(C22-Pad1) -> /AllDrivers/~RESET3
- U7 pad 4: +BATT -> /AllDrivers/Motor5/DECAY
- U7 pad 5: /Motor5/A1 -> /AllDrivers/Motor5/TRQ
- U7 pad 6: GND -> /AllDrivers/Motor5/M1
- U7 pad 7: /Motor5/A2 -> /AllDrivers/Motor5/M0
- U7 pad 8: /Motor5/B2 -> /AllDrivers/Motor5/DIR
- U7 pad 9: GND -> /AllDrivers/Motor5/ENABLE
- U8 pad 1: Net-(C28-Pad1) -> Net-(C11-Pad1)
- U8 pad 10: /Motor3/B1 -> /AllDrivers/MOTOR4_B1
- U8 pad 13: Net-(C27-Pad1) -> Net-(C10-Pad1)
- U8 pad 14: Net-(C26-Pad1) -> Net-(C9-Pad1)
- U8 pad 15: /Motor3/~FAULT -> /AllDrivers/Motor4/~FAULT
- U8 pad 16: Net-(R15-Pad2) -> Net-(R20-Pad2)
- U8 pad 17: /Motor3/~SLEEP -> /AllDrivers/Motor4/~SLEEP
- U8 pad 18: /Motor3/ENABLE -> /AllDrivers/Motor4/ENABLE
- U8 pad 19: STEP3 -> /AllDrivers/STEP4
- U8 pad 2: Net-(C28-Pad2) -> Net-(C11-Pad2)
- U8 pad 20: /Motor3/DIR -> /AllDrivers/Motor4/DIR
- U8 pad 21: /Motor3/M0 -> /AllDrivers/Motor4/M0
- U8 pad 22: /Motor3/M1 -> /AllDrivers/Motor4/M1
- U8 pad 23: /Motor3/TRQ -> /AllDrivers/Motor4/TRQ
- U8 pad 24: /Motor3/DECAY -> (no net)
- U8 pad 3: Net-(C30-Pad1) -> Net-(C13-Pad1)
- U8 pad 5: /Motor3/A1 -> /AllDrivers/MOTOR4_A1
- U8 pad 7: /Motor3/A2 -> /AllDrivers/MOTOR4_A2
- U8 pad 8: /Motor3/B2 -> /AllDrivers/MOTOR4_B2
- U9 pad 1: Net-(C36-Pad1) -> Net-(C19-Pad1)
- U9 pad 10: /Motor2/B1 -> /AllDrivers/MOTOR3_B1
- U9 pad 13: Net-(C35-Pad1) -> Net-(C18-Pad1)
- U9 pad 14: Net-(C34-Pad1) -> Net-(C17-Pad1)
- U9 pad 15: /Motor2/~FAULT -> /AllDrivers/Motor3/~FAULT
- U9 pad 16: Net-(R19-Pad2) -> Net-(R24-Pad2)
- U9 pad 17: /Motor2/~SLEEP -> /AllDrivers/Motor3/~SLEEP
- U9 pad 18: /Motor2/ENABLE -> /AllDrivers/Motor3/ENABLE
- U9 pad 19: STEP2 -> /AllDrivers/STEP3
- U9 pad 2: Net-(C36-Pad2) -> Net-(C19-Pad2)
- U9 pad 20: /Motor2/DIR -> /AllDrivers/Motor3/DIR
- U9 pad 21: /Motor2/M0 -> /AllDrivers/Motor3/M0
- U9 pad 22: /Motor2/M1 -> /AllDrivers/Motor3/M1
- U9 pad 23: /Motor2/TRQ -> /AllDrivers/Motor3/TRQ
- U9 pad 24: /Motor2/DECAY -> /AllDrivers/Motor3/DECAY
- U9 pad 3: Net-(C38-Pad1) -> Net-(C21-Pad1)
- U9 pad 5: /Motor2/A1 -> /AllDrivers/MOTOR3_A1
- U9 pad 7: /Motor2/A2 -> /AllDrivers/MOTOR3_A2
- U9 pad 8: /Motor2/B2 -> /AllDrivers/MOTOR3_B2
Other:
- board size 114.3 x 76.2 mm -> 114.3 x 88.9 mm
- copper layers 2 -> 4

Commit message: new part placements.
Parts:
- removed D1: B340-13-F, footprints:B340-13-F
- removed L1: 100uH, motor_driver:SRR1280A-101M
- removed U2: LM2576SX-3.3, motor_driver:LM2576SX_TO263-5
- added CR1: DPAK_STM, more:LD1117DT33TR, F.Cu at (158.8, 119.0)
- C2: value 100uF -> 0.1uF; footprint Capacitor_SMD:CP_Elec_8x6.2 -> Capacitor_SMD:C_0603_1608Metric_Pad1.08x0.95mm_HandSolder
- C6: value 1000uF -> 10uF; footprint Capacitor_SMD:CP_Elec_8x6.2 -> Capacitor_SMD:C_0805_2012Metric_Pad1.18x1.45mm_HandSolder
- D2: value B340-13-F -> DIODE_SODB340_2P92X4P6_DIO
- moved C47 88.3 mm to (196.2, 99.1), turned to 90 degrees
- moved R6 83.6 mm to (123.8, 96.5)
- moved R8 80.6 mm to (123.8, 99.1)
- moved C43 78.7 mm to (194.3, 108.0)
- moved C44 74.3 mm to (195.6, 118.1), turned to 180 degrees
- moved C45 73.8 mm to (197.5, 106.7), turned to 90 degrees
- moved C46 72.4 mm to (195.6, 113.0), turned to 180 degrees
- moved R10 71.3 mm to (128.3, 95.9)
- moved C12 68.2 mm to (201.9, 71.1), turned to 270 degrees
- moved C42 62.8 mm to (186.1, 95.9), turned to 90 degrees
- moved R12 61.4 mm to (128.3, 99.1)
- moved R1 60.0 mm to (146.7, 100.3)
- moved R7 49.7 mm to (161.9, 97.8)
- moved R2 48.2 mm to (142.2, 99.1)
- moved C41 48.1 mm to (184.2, 95.9), turned to 90 degrees
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Connections:
- C2 pad 1: +BATT -> +12V
- Q1 pad 1: +3V3 -> VCC
- R4 pad 2: +3V3 -> VCC
- U10 pad 24: (no net) -> /AllDrivers/Motor2/DECAY
- U13 pad 24: (no net) -> /AllDrivers/Motor6/DECAY
- U5 pad 13: /AllDrivers/Motor2/TRQ -> /AllDrivers/Motor2/DECAY
- U5 pad 14: /AllDrivers/Motor2/M1 -> /AllDrivers/Motor2/TRQ
- U5 pad 15: /AllDrivers/Motor2/M0 -> /AllDrivers/Motor2/M1
- U5 pad 16: /AllDrivers/Motor2/DIR -> /AllDrivers/Motor2/M0
- U5 pad 17: /AllDrivers/Motor2/ENABLE -> /AllDrivers/Motor2/DIR
- U5 pad 18: /AllDrivers/Motor2/~SLEEP -> /AllDrivers/Motor2/ENABLE
- U5 pad 19: /AllDrivers/Motor2/~FAULT -> /AllDrivers/Motor2/~SLEEP
- U5 pad 20: (no net) -> /AllDrivers/Motor2/~FAULT
- U6 pad 13: /AllDrivers/Motor4/TRQ -> /AllDrivers/Motor4/DECAY
- U6 pad 14: /AllDrivers/Motor4/M1 -> /AllDrivers/Motor4/TRQ
- U6 pad 15: /AllDrivers/Motor4/M0 -> /AllDrivers/Motor4/M1
- U6 pad 16: /AllDrivers/Motor4/DIR -> /AllDrivers/Motor4/M0
- U6 pad 17: /AllDrivers/Motor4/ENABLE -> /AllDrivers/Motor4/DIR
- U6 pad 18: /AllDrivers/Motor4/~SLEEP -> /AllDrivers/Motor4/ENABLE
- U6 pad 19: /AllDrivers/Motor4/~FAULT -> /AllDrivers/Motor4/~SLEEP
- U6 pad 20: (no net) -> /AllDrivers/Motor4/~FAULT
- U7 pad 13: /AllDrivers/Motor6/TRQ -> /AllDrivers/Motor6/DECAY
- U7 pad 14: /AllDrivers/Motor6/M1 -> /AllDrivers/Motor6/TRQ
- U7 pad 15: /AllDrivers/Motor6/M0 -> /AllDrivers/Motor6/M1
- U7 pad 16: /AllDrivers/Motor6/DIR -> /AllDrivers/Motor6/M0
- U7 pad 17: /AllDrivers/Motor6/ENABLE -> /AllDrivers/Motor6/DIR
- U7 pad 18: /AllDrivers/Motor6/~SLEEP -> /AllDrivers/Motor6/ENABLE
- U7 pad 19: /AllDrivers/Motor6/~FAULT -> /AllDrivers/Motor6/~SLEEP
- U7 pad 20: (no net) -> /AllDrivers/Motor6/~FAULT
- U8 pad 24: (no net) -> /AllDrivers/Motor4/DECAY

Commit message: Motor Driver PCB rev 1
Motor Driver PCB rev 1
Parts:
- added H1: MountingHole, MountingHole:MountingHole_3.2mm_M3_ISO14580, F.Cu at (115.6, 115.6)
- added H2: MountingHole, MountingHole:MountingHole_3.2mm_M3_ISO14580, F.Cu at (102.9, 59.7)
- added H3: MountingHole, MountingHole:MountingHole_3.2mm_M3_ISO14580, F.Cu at (181.6, 138.4)
- added H4: MountingHole, MountingHole:MountingHole_3.2mm_M3_ISO14580, F.Cu at (207.0, 59.7)
- CR1: value DPAK_STM -> LD1117DT33TR
- D2: value DIODE_SODB340_2P92X4P6_DIO -> B340-13-F
- moved R9 16.9 mm to (177.4, 93.5), turned to 180 degrees
- moved R2 16.7 mm to (155.2, 109.6), turned to 90 degrees
- moved R7 15.7 mm to (177.4, 95.0), turned to 180 degrees
- moved R11 12.8 mm to (170.7, 93.5)
- moved R1 11.6 mm to (153.7, 109.6), turned to 90 degrees
- moved R3 10.6 mm to (152.1, 109.6), turned to 90 degrees
- moved R8 8.23 mm to (130.3, 94.0), turned to 180 degrees
- moved R16 7.08 mm to (172.1, 110.2), turned to 270 degrees
- moved R6 6.56 mm to (130.3, 95.5), turned to 180 degrees
- moved U4 6.05 mm to (151.1, 102.6), turned to 180 degrees
- moved R12 5.79 mm to (123.7, 95.5)
- moved R13 5.69 mm to (170.7, 95.0)
- moved R14 5.43 mm to (170.6, 117.1), turned to 90 degrees
- moved R17 5.06 mm to (170.6, 110.2), turned to 270 degrees
- moved R10 4.95 mm to (123.7, 94.0)
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Connections:
- J1 pad 1: (no net) -> GND
- J1 pad 10: (no net) -> GND
- J1 pad 12: (no net) -> GND
- J1 pad 15: (no net) -> GND
- J1 pad 16: (no net) -> GND
- J1 pad 17: (no net) -> GND
- J1 pad 18: (no net) -> GND
- J1 pad 2: (no net) -> GND
- J1 pad 22: (no net) -> GND
- J1 pad 23: (no net) -> GND
- J1 pad 24: (no net) -> GND
- J1 pad 26: (no net) -> GND
- J1 pad 27: (no net) -> GND
- J1 pad 28: (no net) -> GND
- J1 pad 32: (no net) -> GND
- J1 pad 33: (no net) -> GND
- J1 pad 35: (no net) -> GND
- J1 pad 36: (no net) -> GND
- J1 pad 37: (no net) -> GND
- J1 pad 38: (no net) -> GND
- J1 pad 4: (no net) -> GND
- J1 pad 40: (no net) -> GND
- J1 pad 7: (no net) -> GND
- J1 pad 8: (no net) -> GND
- U4 pad 10: /AllDrivers/STEP3 -> /AllDrivers/RRef2
- U4 pad 11: /AllDrivers/RRef3 -> /AllDrivers/STEP2
- U4 pad 12: /AllDrivers/STEP4 -> /AllDrivers/STEP1
- U4 pad 13: /AllDrivers/RRef4 -> /AllDrivers/RRef1
- U4 pad 15: /AllDrivers/RRef5 -> /AllDrivers/STEP6
- U4 pad 16: /AllDrivers/STEP5 -> /AllDrivers/RRef6
- U4 pad 17: /AllDrivers/RRef6 -> /AllDrivers/STEP5
- U4 pad 18: /AllDrivers/STEP6 -> /AllDrivers/RRef5
- U4 pad 6: /AllDrivers/STEP1 -> /AllDrivers/RRef4
- U4 pad 7: /AllDrivers/RRef1 -> /AllDrivers/STEP4
- U4 pad 8: /AllDrivers/STEP2 -> /AllDrivers/RRef3
- U4 pad 9: /AllDrivers/RRef2 -> /AllDrivers/STEP3
Routing:
- net GND: track 0.00 -> 199.5 mm, vias 0 -> 128
- net /I2C_SCL: track 0.00 -> 150.4 mm, vias 0 -> 4
- net /I2C_SDA: track 0.00 -> 147.2 mm, vias 0 -> 2
- net +BATT: track 0.00 -> 117.2 mm, vias 0 -> 76
- net /AllDrivers/~INT2: track 0.00 -> 85.0 mm, vias 0 -> 2
- net /AllDrivers/~RESET2: track 0.00 -> 84.5 mm, vias 0 -> 2
- net /AllDrivers/~INT3: track 0.00 -> 83.8 mm, vias 0 -> 2
- net /AllDrivers/~RESET3: track 0.00 -> 81.6 mm, vias 0 -> 2
- net VCC: track 0.00 -> 71.1 mm, vias 0 -> 26
- net /AllDrivers/STEP5: track 0.00 -> 54.7 mm, vias 0 -> 2
- net /AllDrivers/RRef4: track 0.00 -> 54.6 mm, vias 0 -> 2
- net /AllDrivers/STEP6: track 0.00 -> 52.4 mm, vias 0 -> 3
- net /AllDrivers/RRef6: track 0.00 -> 52.4 mm, vias 0 -> 2
- net /AllDrivers/STEP4: track 0.00 -> 50.3 mm, vias 0 -> 2
- net /AllDrivers/STEP1: track 0.00 -> 45.7 mm, vias 0 -> 2
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- added copper zone on F.Cu, net +12V
- added copper zone on F.Cu, net +BATT
- added copper zone on In1.Cu, net +BATT
- added copper zone on F.Cu, net GND
- added copper zone on In2.Cu, net GND
- added copper zone on F.Cu, net VCC
- added copper zone on In1.Cu, net VCC
Other:
- rule via_min_size: 0.4 -> 0.2
- board text added: "Motor Driver board v1.0 g-man"
