File: robarm_pcb/motor_driver/motor_driver_prj/motor_driver_prj.sch (KiCad schematic (older format))
At the start: 9 parts, among them U1 PCA9685PW

Commit message: save
Parts:
- removed C?: 100uF, Capacitor_SMD:CP_Elec_8x6.2, symbol Device:CP1_Small
- removed C?: 1000uF, Capacitor_SMD:CP_Elec_8x6.2, symbol Device:CP1_Small
- removed U?: LM2576HV, motor_driver:LM2576SX_TO263-5, symbol motor_driver:LM2576HV
- added C1, C4: 10uF, Capacitor_SMD:C_0805_2012Metric_Pad1.18x1.45mm_HandSolder, symbol Device:C_Small
- added C2, C3: 100uF, Capacitor_SMD:CP_Elec_8x6.2, symbol Device:CP1_Small
- added C5: 0.1uF, Capacitor_SMD:C_0603_1608Metric_Pad1.08x0.95mm_HandSolder, symbol Device:C_Small
- added C6, C7: 1000uF, Capacitor_SMD:CP_Elec_8x6.2, symbol Device:CP1_Small
- added CR?: LD1117DT33TR, DPAK_STM, symbol LD1117DT33TR:LD1117DT33TR
- added D2: B340-13-F, footprints:B340-13-F, symbol Diode:1N5822
- added L2: 100uH, motor_driver:SRR1280A-101M, symbol Device:L
- added U1: MC78M05_TO252, Package_TO_SOT_SMD:TO-252-2, symbol Regulator_Linear:MC78M05_TO252
- added U2: LM2576SX-3.3, motor_driver:LM2576SX_TO263-5, symbol motor_driver:LM2576SX-3.3
- added U3: LM2576S-12, motor_driver:LM2576SX_TO263-5, symbol motor_driver:LM2576S-12
- D1: value 1N5822 -> B340-13-F; footprint Diode_THT:D_DO-201AD_P15.24mm_Horizontal -> footprints:B340-13-F
- renumbered U1 to U4
Connections:
- net labels added: +12V, +5V, FAN_PWM, I2C_SCL, I2C_SDA
- net labels removed: PWM_SCL, PWM_SDA
- wire segments 64 -> 137
Other:
- note added: "12V to 5V"
- note added: "BATT to 12V conv"
- moved on the sheet: R1, R2, R3, U4

Commit message: new part placements.
Parts:
- removed C2: 100uF, Capacitor_SMD:CP_Elec_8x6.2, symbol Device:CP1_Small
- removed C6: 1000uF, Capacitor_SMD:CP_Elec_8x6.2, symbol Device:CP1_Small
- removed D1: B340-13-F, footprints:B340-13-F, symbol Diode:1N5822
- removed L1: 100uH, motor_driver:SRR1280A-101M, symbol Device:L
- removed U2: LM2576SX-3.3, motor_driver:LM2576SX_TO263-5, symbol motor_driver:LM2576SX-3.3
- added C2: 0.1uF, Capacitor_SMD:C_0603_1608Metric_Pad1.08x0.95mm_HandSolder, symbol Device:C_Small
- added C6: 10uF, Capacitor_SMD:C_0805_2012Metric_Pad1.18x1.45mm_HandSolder, symbol Device:C_Small
- CR1: renamed from CR?; footprint DPAK_STM -> more:LD1117DT33TR
Connections:
- net +12V: now also CR1.2 (VIN), C2.1
- net GND: now also CR1.1 (ADJ/GND), C2.2, C6.2
- net VCC: now also CR1.3 (VOUT), C6.1
Other:
- moved on the sheet: C3, C7, CR1, D2, L2, U3

Commit message: Motor Driver PCB rev 1
Motor Driver PCB rev 1
Connections:
- net AllDrivers/RRef1: now also U4.13 (LED7); no longer U4.7 (LED1)
- net AllDrivers/RRef2: now also U4.10 (LED4); no longer U4.9 (LED3)
- net AllDrivers/RRef3: now also U4.8 (LED2); no longer U4.11 (LED5)
- net AllDrivers/RRef4: now also U4.6 (LED0); no longer U4.13 (LED7)
- net AllDrivers/RRef5: now also U4.18 (LED11); no longer U4.15 (LED8)
- net AllDrivers/RRef6: now also U4.16 (LED9); no longer U4.17 (LED10)
- net AllDrivers/STEP1: now also U4.12 (LED6); no longer U4.6 (LED0)
- net AllDrivers/STEP2: now also U4.11 (LED5); no longer U4.8 (LED2)
- net AllDrivers/STEP3: now also U4.9 (LED3); no longer U4.10 (LED4)
- net AllDrivers/STEP4: now also U4.7 (LED1); no longer U4.12 (LED6)
- net AllDrivers/STEP5: now also U4.17 (LED10); no longer U4.16 (LED9)
- net AllDrivers/STEP6: now also U4.15 (LED8); no longer U4.18 (LED11)
