File: robarm_pcb/motor_driver/motor_driver_prj/single_driver.sch (KiCad schematic (older format))
At the start: 13 parts, among them U5 DRV8886PWPR‎

Commit message: save
Parts:
- renumbered C3 to C10, C4 to C11, C5 to C12, C6 to C13, C7 to C14, C8 to C15, C1 to C8, C2 to C9, R16 to R18, R17 to R19, R18 to R20, R19 to R21, U5 to U8

Commit message: new part placements.
Changed lines of the file:
@@
 $Descr A4 11693 8268
 encoding utf-8
-Sheet 14 15
+Sheet 15 15
 Title ""
 Date ""
@@
 AR Path="/603463D6/603659BE/6024ACA6" Ref="U10"  Part="1"
 AR Path="/603463D6/603659CE/6024ACA6" Ref="U11"  Part="1"
-F 0 "U12" H 5400 4600 50  0000 C CNN
+F 0 "U13" H 5400 4600 50  0000 C CNN
 F 1 "DRV8886PWPR‎" H 5900 3100 50  0000 C CNN
 F 2 "motor_driver:DRV8886_HTSSOP-24" H 5400 4600 50  0001 C CNN
@@
 AR Path="/603463D6/603659BE/60251CEA" Ref="C27"  Part="1"
 AR Path="/603463D6/603659CE/60251CEA" Ref="C35"  Part="1"
-F 0 "C43" H 6642 3296 50  0000 L CNN
+F 0 "C51" H 6642 3296 50  0000 L CNN
 F 1 "0.022uF" H 6642 3205 50  0000 L CNN
 F 2 "Capacitor_SMD:C_0603_1608Metric_Pad1.08x0.95mm_HandSolder" H 6550 3250 50  0001 C CNN
@@
 AR Path="/603463D6/603659BE/602523CC" Ref="C29"  Part="1"
 AR Path="/603463D6/603659CE/602523CC" Ref="C37"  Part="1"
-F 0 "C45" H 6892 3496 50  0000 L CNN
+F 0 "C53" H 6892 3496 50  0000 L CNN
 F 1 "0.22uF" H 6892 3405 50  0000 L CNN
 F 2 "Capacitor_SMD:C_0603_1608Metric_Pad1.08x0.95mm_HandSolder" H 6800 3450 50  0001 C CNN
@@
 AR Path="/603463D6/603659BE/60253DDB" Ref="C25"  Part="1"
 AR Path="/603463D6/603659CE/60253DDB" Ref="C33"  Part="1"
-F 0 "C41" H 4500 4650 50  0000 L CNN
+F 0 "C49" H 4500 4650 50  0000 L CNN
 F 1 "0.47uF" H 4500 4550 50  0000 L CNN
 F 2 "Capacitor_SMD:C_0805_2012Metric_Pad1.18x1.45mm_HandSolder" H 4750 4600 50  0001 C CNN
@@
 AR Path="/603463D6/603659BE/602546D2" Ref="C26"  Part="1"
 AR Path="/603463D6/603659CE/602546D2" Ref="C34"  Part="1"
-F 0 "C42" H 5092 4646 50  0000 L CNN
+F 0 "C50" H 5092 4646 50  0000 L CNN
 F 1 "0.47uF" H 5092 4555 50  0000 L CNN
 F 2 "Capacitor_SMD:C_0805_2012Metric_Pad1.18x1.45mm_HandSolder" H 5000 4600 50  0001 C CNN
@@
 AR Path="/603463D6/603659BE/6025A5DA" Ref="C30"  Part="1"
 AR Path="/603463D6/603659CE/6025A5DA" Ref="C38"  Part="1"
-F 0 "C46" H 7241 4496 50  0000 L CNN
+F 0 "C54" H 7241 4496 50  0000 L CNN
 F 1 "100uF" H 7241 4405 50  0000 L CNN
 F 2 "Capacitor_SMD:CP_Elec_8x6.2" H 7150 4450 50  0001 C CNN
@@
 AR Path="/603463D6/603659BE/6025C5BE" Ref="C28"  Part="1"
 AR Path="/603463D6/603659CE/6025C5BE" Ref="C36"  Part="1"
-F 0 "C44" H 6792 4496 50  0000 L CNN
+F 0 "C52" H 6792 4496 50  0000 L CNN
 F 1 "0.01uF" H 6792 4405 50  0000 L CNN
 F 2 "Capacitor_SMD:C_0603_1608Metric_Pad1.08x0.95mm_HandSolder" H 6700 4450 50  0001 C CNN
@@
 AR Path="/603463D6/603659BE/6025CAB5" Ref="#PWR058"  Part="1"
 AR Path="/603463D6/603659CE/6025CAB5" Ref="#PWR067"  Part="1"
-F 0 "#PWR076" H 7500 3750 50  0001 C CNN
+F 0 "#PWR085" H 7500 3750 50  0001 C CNN
 F 1 "GND" H 7505 3827 50  0000 C CNN
 F 2 "" H 7500 4000 50  0001 C CNN
@@
 AR Path="/603463D6/603659BE/6028F28B" Ref="#PWR054"  Part="1"
 AR Path="/603463D6/603659CE/6028F28B" Ref="#PWR063"  Part="1"
-F 0 "#PWR072" H 6400 4500 50  0001 C CNN
+F 0 "#PWR081" H 6400 4500 50  0001 C CNN
 F 1 "GND" H 6405 4577 50  0000 C CNN
 F 2 "" H 6400 4750 50  0001 C CNN
@@
 AR Path="/603463D6/603659BE/60294232" Ref="#PWR056"  Part="1"
 AR Path="/603463D6/603659CE/60294232" Ref="#PWR065"  Part="1"
-F 0 "#PWR074" H 7150 4500 50  0001 C CNN
+F 0 "#PWR083" H 7150 4500 50  0001 C CNN
 F 1 "GND" H 7155 4577 50  0000 C CNN
 F 2 "" H 7150 4750 50  0001 C CNN
@@
 AR Path="/603463D6/603659BE/602DD586" Ref="#PWR053"  Part="1"
 AR Path="/603463D6/603659CE/602DD586" Ref="#PWR062"  Part="1"
-F 0 "#PWR071" H 5000 4500 50  0001 C CNN
+F 0 "#PWR080" H 5000 4500 50  0001 C CNN
 F 1 "GND" H 5005 4577 50  0000 C CNN
 F 2 "" H 5000 4750 50  0001 C CNN
@@
 AR Path="/603463D6/603659BE/602E5BBF" Ref="#PWR052"  Part="1"
 AR Path="/603463D6/603659CE/602E5BBF" Ref="#PWR061"  Part="1"
-F 0 "#PWR070" H 4750 4500 50  0001 C CNN
+F 0 "#PWR079" H 4750 4500 50  0001 C CNN
 F 1 "GND" H 4755 4577 50  0000 C CNN
 F 2 "" H 4750 4750 50  0001 C CNN
@@
 AR Path="/603463D6/603659BE/602E723F" Ref="R28"  Part="1"
 AR Path="/603463D6/603659CE/602E723F" Ref="R32"  Part="1"
-F 0 "R36" V 4563 4050 50  0000 C CNN
+F 0 "R40" V 4563 4050 50  0000 C CNN
 F 1 "rref" H 4518 4005 50  0001 L CNN
 F 2 "Resistor_SMD:R_0603_1608Metric_Pad0.98x0.95mm_HandSolder" H 4450 4050 50  0001 C CNN
@@
 AR Path="/603463D6/603659BE/602E7D4F" Ref="R26"  Part="1"
 AR Path="/603463D6/603659CE/602E7D4F" Ref="R30"  Part="1"
-F 0 "R34" H 3618 4200 50  0000 L CNN
+F 0 "R38" H 3618 4200 50  0000 L CNN
 F 1 "R_Small_US" H 3618 4155 50  0001 L CNN
 F 2 "Resistor_SMD:R_0603_1608Metric_Pad0.98x0.95mm_HandSolder" H 3550 4200 50  0001 C CNN
@@
 AR Path="/603463D6/603659BE/602E8822" Ref="R27"  Part="1"
 AR Path="/603463D6/603659CE/602E8822" Ref="R31"  Part="1"
-F 0 "R35" H 3618 4550 50  0000 L CNN
+F 0 "R39" H 3618 4550 50  0000 L CNN
 F 1 "R_Small_US" H 3618 4505 50  0001 L CNN
 F 2 "Resistor_SMD:R_0603_1608Metric_Pad0.98x0.95mm_HandSolder" H 3550 4550 50  0001 C CNN
@@
 AR Path="/603463D6/603659BE/602E9389" Ref="C24"  Part="1"
 AR Path="/603463D6/603659CE/602E9389" Ref="C32"  Part="1"
-F 0 "C40" H 4092 4596 50  0000 L CNN
+F 0 "C48" H 4092 4596 50  0000 L CNN
 F 1 "0.1uF" H 4092 4505 50  0000 L CNN
 F 2 "Capacitor_SMD:C_0603_1608Metric_Pad1.08x0.95mm_HandSolder" H 4000 4550 50  0001 C CNN
@@
 AR Path="/603463D6/603659BE/602EE5D1" Ref="#PWR051"  Part="1"
 AR Path="/603463D6/603659CE/602EE5D1" Ref="#PWR060"  Part="1"
-F 0 "#PWR069" H 4000 4500 50  0001 C CNN
+F 0 "#PWR078" H 4000 4500 50  0001 C CNN
 F 1 "GND" H 4005 4577 50  0000 C CNN
 F 2 "" H 4000 4750 50  0001 C CNN
@@
 AR Path="/603463D6/603659BE/602EF163" Ref="#PWR050"  Part="1"
 AR Path="/603463D6/603659CE/602EF163" Ref="#PWR059"  Part="1"
-F 0 "#PWR068" H 3550 4500 50  0001 C CNN
+F 0 "#PWR077" H 3550 4500 50  0001 C CNN
 F 1 "GND" H 3555 4577 50  0000 C CNN
 F 2 "" H 3550 4750 50  0001 C CNN
@@
 AR Path="/603463D6/603659BE/602E14BD" Ref="R29"  Part="1"
 AR Path="/603463D6/603659CE/602E14BD" Ref="R33"  Part="1"
-F 0 "R37" H 4818 4300 50  0000 L CNN
+F 0 "R41" H 4818 4300 50  0000 L CNN
 F 1 "R_Small_US" H 4818 4255 50  0001 L CNN
 F 2 "Resistor_SMD:R_0603_1608Metric_Pad0.98x0.95mm_HandSolder" H 4750 4300 50  0001 C CNN
@@
 AR Path="/603463D6/603659BE/604AB47A" Ref="#PWR057"  Part="1"
 AR Path="/603463D6/6036598E/604AB47A" Ref="#PWR084"  Part="1"
-F 0 "#PWR075" H 7500 3350 50  0001 C CNN
+F 0 "#PWR084" H 7500 3350 50  0001 C CNN
 F 1 "+BATT" H 7515 3673 50  0000 C CNN
 F 2 "" H 7500 3500 50  0001 C CNN
@@
 AR Path="/603463D6/603659BE/604AC0D3" Ref="#PWR055"  Part="1"
 AR Path="/603463D6/6036598E/604AC0D3" Ref="#PWR082"  Part="1"
-F 0 "#PWR073" H 7150 4050 50  0001 C CNN
+F 0 "#PWR082" H 7150 4050 50  0001 C CNN
 F 1 "+BATT" H 7165 4373 50  0000 C CNN
 F 2 "" H 7150 4200 50  0001 C CNN
@@
 AR Path="/603463D6/603659BE/602532B9" Ref="C31"  Part="1"
 AR Path="/603463D6/603659CE/602532B9" Ref="C39"  Part="1"
-F 0 "C47" H 7592 3846 50  0000 L CNN
+F 0 "C55" H 7592 3846 50  0000 L CNN
 F 1 "0.01uF" H 7592 3755 50  0000 L CNN
 F 2 "Capacitor_SMD:C_0603_1608Metric_Pad1.08x0.95mm_HandSolder" H 7500 3800 50  0001 C CNN
