Commit message: working 3 joint arm

File: robarm_code/src/robarm_description/urdf/robarm.urdf.xacro (robot description, xacro)
@@ -8,8 +8,8 @@
       <type>transmission_interface/SimpleTransmission</type>
       <joint name="${joint}">
-        <hardwareInterface>hardware_interface/PositionJointInterface</hardwareInterface>
+        <hardwareInterface>hardware_interface/EffortJointInterface</hardwareInterface>
       </joint>
       <actuator name="motor${n}">
-        <hardwareInterface>hardware_interface/PositionJointInterface</hardwareInterface>
+        <hardwareInterface>hardware_interface/EffortJointInterface</hardwareInterface>
         <mechanicalReduction>1</mechanicalReduction>
       </actuator>
@@ -36,5 +36,5 @@
     </visual>
     <collision>
-      <origin xyz="0 0 0" rpy="0 0 0"/>
+      <origin xyz="0 0 0.1" rpy="0 0 0"/>
       <geometry>
         <cylinder radius="0.4" length="0.2"/>
@@ -43,9 +43,9 @@
     <!-- inertia is not correct - change this later -->
     <inertial>
-      <origin xyz="0 0 0" />
+      <!-- <origin xyz="0 0 0" /> -->
       <mass value="0.1" />
-      <inertia ixx="0.1" ixy="0.0" ixz="0.0"
-               iyy="0.1" iyz="0.0"
-               izz="0.1" />
+      <inertia ixx="0.001" ixy="0.0" ixz="0.0"
+               iyy="0.001" iyz="0.0"
+               izz="0.001" />
     </inertial>
   </link>
@@ -76,9 +76,9 @@
     </collision>
    <inertial>
-      <origin xyz="0 0 0" />
+      <!-- <origin xyz="0 0 0" /> -->
       <mass value="0.1" />
-      <inertia ixx="0.1" ixy="0.0" ixz="0.0"
-               iyy="0.1" iyz="0.0"
-               izz="0.1" />
+      <inertia ixx="0.001" ixy="0.0" ixz="0.0"
+               iyy="0.001" iyz="0.0"
+               izz="0.001" />
     </inertial>
   </link>
@@ -109,9 +109,9 @@
     </collision>
    <inertial>
-      <origin xyz="0 0 0" />
+      <!-- <origin xyz="0 0 0" /> -->
       <mass value="0.1" />
-      <inertia ixx="0.1" ixy="0.0" ixz="0.0"
-               iyy="0.1" iyz="0.0"
-               izz="0.1" />
+      <inertia ixx="0.001" ixy="0.0" ixz="0.0"
+               iyy="0.001" iyz="0.0"
+               izz="0.001" />
     </inertial>
   </link>
@@ -142,10 +142,16 @@
     </collision>
    <inertial>
-      <origin xyz="0 0 0" />
+      <!-- <origin xyz="0 0 0" /> -->
       <mass value="0.1" />
-      <inertia ixx="0.1" ixy="0.0" ixz="0.0"
-               iyy="0.1" iyz="0.0"
-               izz="0.1" />
+      <inertia ixx="0.00" ixy="0.0" ixz="0.0"
+               iyy="0.001" iyz="0.0"
+               izz="0.001" />
     </inertial>
   </link>
+  <gazebo>
+    <plugin name="gazebo_ros_control" filename="libgazebo_ros_control.so">
+      <robotNamespace>/robarm</robotNamespace>
+      <robotSimType>gazebo_ros_control/DefaultRobotHWSim</robotSimType>
+    </plugin>
+  </gazebo>
 </robot>
